File: pcb/52Te_Rev.kicad_pcb (KiCad board)
At the start: 2 copper layers, 159.1 x 145.6 mm, 62 parts, among them J1 MJ-4PP-9, J2 Conn_01x04, SW1 SW_PUSH, SW10 SW_PUSH, SW11 SW_PUSH, SW12 SW_PUSH, SW13 SW_PUSH, SW14 SW_PUSH, SW15 SW_PUSH, SW16 SW_PUSH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

Commit message: latest 20190201
Parts:
- added G***: LOGO, 52Te_Rev:karin, F.Cu at (196.6, 126.5)
Other:
- board text added: "52Te Split Keyboard PCB by @SA_EndlessGame"

Commit message: 20190213 added logos
Parts:
- removed the G*** at (196.6, 126.5)
- added G***: LOGO, 52Te_Rev:emptystringLogo, B.Cu at (186.3, 134.1)
- added G***: LOGO, 52Te_Rev:52TeLogo, F.Cu at (193.2, 131.1)
Other:
- board text added: "52Te Split Keyboard by emptystring @SA_EndlessGame"
- board text removed: "52Te Split Keyboard PCB by @SA_EndlessGame"
